File: KiCad/IC-705 Audio Interface.kicad_pcb (KiCad board)
At the start: 2 copper layers, 36.2 x 21.8 mm, 11 parts, among them J1 Conn_01x02, J2 Conn_01x02, J3 Conn_01x02, J4 Conn_01x02, T1 SM-LP-5001, T2 SM-LP-5001

Commit message: Change text and remove tracks inside pads.
Other:
- board text added: "IC-705 Audio Interface N1CDV project802.net"
- board text removed: "Audio Interface N1CDV project802.net"
Changed lines of the file:
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@@
 		(capping no)
 		(filling no)
-		(zone_defaults)
 		(pcbplotparams
 			(layerselection 0x00000000_00000000_55555555_5755f5ff)
@@
 		(layer "F.Cu")
 		(at 131.25 82 -90)
+		(property "Reference" "R4"
+			(at 0 -1.25 90)
+			(unlocked yes)
+			(layer "F.SilkS")
+			(effects
+				(font
+					(size 1 1)
+					(thickness 0.15)
+				)
+			)
+		)
 		(property "Value" "~"
 			(at 0 1 270)
@@
 			(layer "F.Fab")
 			(hide yes)
-			(effects
-				(font
-					(size 1 1)
-					(thickness 0.15)
-				)
-			)
-		)
-		(property "Reference" "R4"
-			(at 0 -1.25 90)
-			(unlocked yes)
-			(layer "F.SilkS")
 			(effects
 				(font
@@
 		(layer "F.Cu")
 		(at 133.25 71.744114 -90)
+		(property "Reference" "R1"
+			(at -0.044276 -1.25 90)
+			(unlocked yes)
+			(layer "F.SilkS")
+			(effects
+				(font
+					(size 1 1)
+					(thickness 0.15)
+				)
+			)
+		)
 		(property "Value" "~"
 			(at 0 1 270)
@@
 			(layer "F.Fab")
 			(hide yes)
-			(effects
-				(font
-					(size 1 1)
-					(thickness 0.15)
-				)
-			)
-		)
-		(property "Reference" "R1"
-			(at -0.044276 -1.25 90)
-			(unlocked yes)
-			(layer "F.SilkS")
 			(effects
 				(font
@@
 		)
 	)
-	(gr_text "Audio Interface\nN1CDV\nproject802.net"
-		(at 121.5 77.75 0)
+	(gr_text "IC-705 Audio Interface\nN1CDV\nproject802.net"
+		(at 119.75 77.75 0)
 		(layer "B.SilkS")
 		(effects
@@
 	)
 	(segment
-		(start 124.254276 74.294276)
-		(end 124.25 74.29)
-		(width 0.6)
-		(layer "F.Cu")
-		(net "/COMP_MIC_SH")
-	)
-	(segment
-		(start 124.295886 74.244114)
-		(end 124.25 74.29)
-		(width 0.6)
-		(layer "F.Cu")
-		(net "/COMP_MIC_SH")
+		(start 112.25 69.21)
+		(end 108.015 69.21)
+		(width 0.6)
+		(layer "F.Cu")
+		(net "/705_SP")
+	)
+	(segment
+		(start 108.015 69.21)
+		(end 106.75 70.475)
+		(width 0.6)
+		(layer "F.Cu")
+		(net "/705_SP")
+	)
+	(segment
+		(start 108.025 74.29)
+		(end 106.75 73.015)
+		(width 0.6)
+		(layer "F.Cu")
+		(net "/705_SP_SH")
+	)
+	(segment
+		(start 112.25 74.29)
+		(end 108.025 74.29)
+		(width 0.6)
+		(layer "F.Cu")
+		(net "/705_SP_SH")
 	)
 	(segment
@@
 	)
 	(segment
+		(start 125 67.5)
+		(end 127.3375 67.5)
+		(width 0.6)
+		(layer "F.Cu")
+		(net "Net-(R2-Pad1)")
+	)
+	(segment
+		(start 124.25 69.21)
+		(end 124.25 68.25)
+		(width 0.6)
+		(layer "F.Cu")
+		(net "Net-(R2-Pad1)")
+	)
+	(segment
+		(start 124.25 68.25)
+		(end 125 67.5)
+		(width 0.6)
+		(layer "F.Cu")
+		(net "Net-(R2-Pad1)")
+	)
+	(segment
+		(start 132 69)
+		(end 130.5 67.5)
+		(width 0.6)
+		(layer "F.Cu")
+		(net "Net-(R1-Pad2)")
+	)
+	(segment
+		(start 130.5 67.5)
+		(end 129.1625 67.5)
+		(width 0.6)
+		(layer "F.Cu")
+		(net "Net-(R1-Pad2)")
+	)
+	(segment
+		(start 132 71.744114)
+		(end 132 69)
+		(width 0.6)
+		(layer "F.Cu")
+		(net "Net-(R1-Pad2)")
+	)
+	(segment
 		(start 137.225 70.475)
 		(end 135.994114 69.244114)
@@
 	)
 	(segment
-		(start 132 69)
-		(end 130.5 67.5)
-		(width 0.6)
-		(layer "F.Cu")
-		(net "Net-(R1-Pad2)")
-	)
-	(segment
-		(start 130.5 67.5)
-		(end 129.1625 67.5)
-		(width 0.6)
-		(layer "F.Cu")
-		(net "Net-(R1-Pad2)")
-	)
-	(segment
-		(start 132 71.744114)
-		(end 132 69)
-		(width 0.6)
-		(layer "F.Cu")
-		(net "Net-(R1-Pad2)")
-	)
-	(segment
-		(start 125 67.5)
-		(end 127.3375 67.5)
-		(width 0.6)
-		(layer "F.Cu")
-		(net "Net-(R2-Pad1)")
-	)
-	(segment
-		(start 124.25 69.21)
-		(end 124.25 68.25)
-		(width 0.6)
-		(layer "F.Cu")
-		(net "Net-(R2-Pad1)")
-	)
-	(segment
-		(start 124.25 68.25)
-		(end 125 67.5)
-		(width 0.6)
-		(layer "F.Cu")
-		(net "Net-(R2-Pad1)")
-	)
-	(segment
-		(start 132.504444 84.504444)
-		(end 132.5 84.5)
-		(width 0.6)
-		(layer "F.Cu")
-		(net "/COMP_SP_SH")
-	)
-	(segment
-		(start 124.29 84.5)
-		(end 124.25 84.54)
-		(width 0.6)
-		(layer "F.Cu")
-		(net "/COMP_SP_SH")
+		(start 139.165941 84.504444)
+		(end 139.165941 79.503441)
+		(width 0.6)
+		(layer "F.Cu")
+		(net "/COMP_SP")
 	)
 	(segment
@@
 	)
 	(segment
-		(start 108.025 74.29)
-		(end 106.75 73.015)
-		(width 0.6)
-		(layer "F.Cu")
-		(net "/705_SP_SH")
-	)
-	(segment
-		(start 112.25 74.29)
-		(end 108.025 74.29)
-		(width 0.6)
-		(layer "F.Cu")
-		(net "/705_SP_SH")
-	)
-	(segment
-		(start 112.25 69.21)
-		(end 108.015 69.21)
-		(width 0.6)
-		(layer "F.Cu")
-		(net "/705_SP")
-	)
-	(segment
-		(start 108.015 69.21)
-		(end 106.75 70.475)
-		(width 0.6)
-		(layer "F.Cu")
-		(net "/705_SP")
+		(start 137.3375 79.5)
+		(end 132.5 79.5)
+		(width 0.6)
+		(layer "F.Cu")
+		(net "Net-(R3-Pad1)")
+	)
+	(segment
+		(start 124.25 79.46)
+		(end 127.46 79.46)
+		(width 0.6)
+		(layer "F.Cu")
+		(net "Net-(R4-Pad2)")
+	)
+	(segment
+		(start 127.46 79.46)
+		(end 130 82)
+		(width 0.6)
+		(layer "F.Cu")
+		(net "Net-(R4-Pad2)")
 	)
 	(segment
@@
 		(net "/705_MIC_SH")
 	)
-	(segment
-		(start 139.165941 84.504444)
-		(end 139.165941 79.503441)
-		(width 0.6)
-		(layer "F.Cu")
-		(net "/COMP_SP")
-	)
-	(segment
-		(start 139.165941 79.503441)
-		(end 139.1625 79.5)
-		(width 0.6)
-		(layer "F.Cu")
-		(net "/COMP_SP")
-	)
-	(segment
-		(start 132.01 79.53)
-		(end 132 79.52)
-		(width 0.6)
-		(layer "F.Cu")
-		(net "Net-(R3-Pad1)")
-	)
-	(segment
-		(start 137.3375 79.5)
-		(end 132.5 79.5)
-		(width 0.6)
-		(layer "F.Cu")
-		(net "Net-(R3-Pad1)")
-	)
-	(segment
-		(start 124.25 79.46)
-		(end 127.46 79.46)
-		(width 0.6)
-		(layer "F.Cu")
-		(net "Net-(R4-Pad2)")
-	)
-	(segment
-		(start 127.46 79.46)
-		(end 130 82)
-		(width 0.6)
-		(layer "F.Cu")
-		(net "Net-(R4-Pad2)")
-	)
 	(group ""
