File: KiCad/IC-705 Audio Interface.kicad_sch (KiCad schematic)
At the start: 11 parts, among them J1 Conn_01x02, J2 Conn_01x02, J3 Conn_01x02, J4 Conn_01x02, T1 SM-LP-5001, T2 SM-LP-5001

Commit message: Add audio jacks
Parts:
- added C1: 0.1uF, symbol Device:C
- added J5, J6: AudioPlug4, symbol Connector_Audio:AudioPlug4
- added J7: AudioPlug3, symbol Connector_Audio:AudioPlug3
- J1, J2, J3, J4: now fitted; now left out of the parts list
Connections:
- net 705_MIC: now also C1.2
- net 705_MIC_SH: now also J5.S
- net 705_SP: now also J7.T
- net 705_SP_SH: now also J7.S
- net COMP_MIC: now also J6.T
- net COMP_SP: now also J6.R1
- net COMP_SP_SH: now also J6.S
- new net: C1.1, J5.T

Commit message: Update connector names
Parts:
- J5: value AudioPlug4 -> 2.5mm TRRS
- J6: value AudioPlug4 -> 3.5mm TRRS
- J7: value AudioPlug3 -> 3.5mm TRS
Changed lines of the file:
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@@
 			)
 		)
-		(property "Value" "AudioPlug4"
+		(property "Value" "3.5mm TRRS"
 			(at 261.62 93.9799 0)
 			(show_name no)
@@
 			)
 		)
-		(property "Value" "AudioPlug4"
+		(property "Value" "2.5mm TRRS"
 			(at 54.61 99.06 0)
 			(show_name no)
@@
 		(dnp no)
 		(property "Reference" "J7"
-			(at 54.61 91.44 0)
-			(show_name no)
-			(do_not_autoplace no)
-			(effects
-				(font
-					(size 1.27 1.27)
-				)
-			)
-		)
-		(property "Value" "AudioPlug3"
-			(at 54.61 88.9 0)
-			(show_name no)
-			(do_not_autoplace no)
+			(at 54.61 71.12 0)
+			(show_name no)
+			(do_not_autoplace no)
+			(effects
+				(font
+					(size 1.27 1.27)
+				)
+			)
+		)
+		(property "Value" "3.5mm TRS"
+			(at 54.61 73.66 0)
+			(show_name no)
+			(do_not_autoplace no)

Commit message: Add link to GitHub repo
Other:
- note added: "https://github.com/project802/ic-705_audio_interface"
Changed lines of the file:
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@@
 	(generator_version "10.0")
 	(paper "A4")
+	(text "https://github.com/project802/ic-705_audio_interface"
+		(exclude_from_sim no)
+		(at 231.902 173.99 0)
+		(effects
+			(font
+				(size 1.778 1.778)
+			)
+		)
+	)
 	(junction
 		(at 101.6 80.01)
